Commit message: Try to add go1 support

File: src/data/a1.urdf (robot description, URDF)
Before this commit: robot a1_description, 18 links, 17 joints
Links:
- link FL_hip: geometry collision cylinder length=0.04 radius=0.046; visual mesh filename=a1_meshes/hip.obj scale=1 1 1
- link FL_lower: geometry collision box size=0.2 0.016 0.016; visual mesh filename=a1_meshes/calf.obj scale=1 1 1
- link FL_upper: geometry collision box size=0.2 0.0245 0.034; visual mesh filename=a1_meshes/thigh.obj scale=1 1 1
- link FR_hip: geometry collision cylinder length=0.04 radius=0.046; visual mesh filename=a1_meshes/hip.obj scale=1 1 1
- link FR_lower: geometry collision box size=0.2 0.016 0.016; visual mesh filename=a1_meshes/calf.obj scale=1 1 1
- link FR_upper: geometry collision box size=0.2 0.0245 0.034; visual mesh filename=a1_meshes/thigh_mirror.obj scale=1 1 1
- link RL_hip: geometry collision cylinder length=0.04 radius=0.046; visual mesh filename=a1_meshes/hip.obj scale=1 1 1
- link RL_lower: geometry collision box size=0.2 0.016 0.016; visual mesh filename=a1_meshes/calf.obj scale=1 1 1
- link RL_upper: geometry collision box size=0.2 0.0245 0.034; visual mesh filename=a1_meshes/thigh.obj scale=1 1 1
- link RR_hip: geometry collision cylinder length=0.04 radius=0.046; visual mesh filename=a1_meshes/hip.obj scale=1 1 1
- link RR_lower: geometry collision box size=0.2 0.016 0.016; visual mesh filename=a1_meshes/calf.obj scale=1 1 1
- link RR_upper: geometry collision box size=0.2 0.0245 0.034; visual mesh filename=a1_meshes/thigh_mirror.obj scale=1 1 1
- link trunk: geometry collision box size=0.267 0.194 0.114; visual mesh filename=a1_meshes/trunk.obj scale=1 1 1
